File: Regulator/Regulator.kicad_pcb (KiCad board)
At the start: 2 copper layers, 6 parts, among them U1 LMR16006YQ3

Commit message: Finish off PCB for this
Parts:
- added J1: Conn_01x04, Connector_PinHeader_2.54mm:PinHeader_1x04_P2.54mm_Vertical, B.Cu at (166.4, 69.7)
- added Logo1: AJK, RevK:AJK, B.Cu at (163.7, 61.5)
- added R1: 10M 1% or 0R, RevK:R_0603, F.Cu at (159.1, 66.9)
- added R2: 1.8M 1% or NF, RevK:R_0603, F.Cu at (165.5, 66.3)
- U1: value LMR16006YQ3 -> LMR16006+FB; footprint RevK:RegulatorBlock -> RevK:RegulatorBlockFB
- moved C1 179.6 mm to (166.0, 63.4)
- moved U1 175.8 mm to (163.9, 63.6), turned to 180 degrees
- moved C2 175.0 mm to (164.7, 60.1)
- moved D1 169.3 mm to (161.6, 60.4)
- moved L1 168.6 mm to (160.0, 63.6), turned to 180 degrees
- moved C3 163.2 mm to (158.5, 60.1)
Connections:
- U1 pad 3: Net-(U1-Pad3) -> GND
Routing:
- net Net-(J1-Pad2): track 0.00 -> 13.7 mm
- net Net-(J1-Pad1): track 0.00 -> 10.5 mm, vias 0 -> 1
- net Net-(R1-Pad2): track 0.00 -> 9.35 mm
- net Net-(J1-Pad4): track 0.00 -> 6.31 mm
- net GND: track 0.00 -> 3.14 mm, vias 0 -> 1
- added copper zone on B.Cu, net GND
- added copper zone on F.Cu, net GND
Other:
- board outline added: 10.2 x 12.7 mm
- net class Default removed
- board text added: "GND"
- board text added: "SHDN"
- board text added: "VIN"
- board text added: "VOUT"

Commit message: Reverse
Parts:
- J1: moved to F.Cu
- moved R1 10.0 mm to (165.3, 59.0), turned to 180 degrees
- moved C3 9.50 mm to (166.0, 65.9)
- moved R2 9.29 mm to (159.0, 59.7), turned to 180 degrees
- moved C2 7.70 mm to (159.7, 65.9)
- moved J1 7.62 mm to (158.8, 69.8)
- moved C1 7.56 mm to (158.5, 62.6)
- moved D1 5.23 mm to (162.8, 65.5)
- moved L1 4.66 mm to (164.5, 62.4)
- moved U1 3.54 mm to (160.6, 62.4), turned to 0 degrees
- moved Logo1 1.74 mm to (162.0, 61.5)
Routing:
- net Net-(J1-Pad2): track 13.7 -> 7.41 mm
- net Net-(J1-Pad4): track 6.31 -> 12.1 mm
- net Net-(J1-Pad1): track 10.5 -> 7.98 mm, vias 1 -> 0

Commit message: Library update
Other:
- outline, holes or cut-outs redrawn
- board text added: "www.me.uk"
- board text added: "↑"
- board text added: "↓"
- board text added: "⏚"
Changed lines of the file:
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@@
     )
   )
-  (footprint "Connector_PinHeader_2.54mm:PinHeader_1x04_P2.54mm_Vertical" (layer "F.Cu")
+  (footprint "Connector_PinHeader_2.54mm:PinHeader_1x04_P2.54mm_Vertical" locked (layer "F.Cu")
     (at 158.75 69.85 90)
     (descr "Through hole straight pin header, 1x04, 2.54mm pitch, single row")
@@
     (fp_line (start 1.27 8.89) (end -1.27 8.89) (layer "F.Fab") (width 0.1))
     (fp_line (start 1.27 -1.27) (end 1.27 8.89) (layer "F.Fab") (width 0.1))
-    (pad "1" thru_hole circle (at 0 0 90) (size 1.7 1.7) (drill 1) (layers *.Cu *.Mask)
+    (pad "1" smd rect locked (at -0.635 0 90) (size 1.27 1.7) (layers "B.Cu" "B.Mask")
       (net 1 "Net-(J1-Pad1)") (pinfunction "Pin_1") (pintype "passive"))
-    (pad "2" thru_hole oval (at 0 2.54 90) (size 1.7 1.7) (drill 1) (layers *.Cu *.Mask)
+    (pad "1" thru_hole circle locked (at 0 0 90) (size 1.7 1.7) (drill 1) (layers *.Cu *.Mask)
+      (net 1 "Net-(J1-Pad1)") (pinfunction "Pin_1") (pintype "passive"))
+    (pad "1" smd rect locked (at -0.635 0 90) (size 1.27 1.7) (layers "F.Cu" "F.Mask")
+      (net 1 "Net-(J1-Pad1)") (pinfunction "Pin_1") (pintype "passive"))
+    (pad "2" smd rect locked (at -0.635 2.54 90) (size 1.27 1.7) (layers "B.Cu" "B.Mask")
       (net 2 "Net-(J1-Pad2)") (pinfunction "Pin_2") (pintype "passive"))
-    (pad "3" thru_hole roundrect (at 0 5.08 90) (size 1.7 1.7) (drill 1) (layers *.Cu *.Mask) (roundrect_rratio 0.25)
+    (pad "2" smd rect locked (at -0.635 2.54 90) (size 1.27 1.7) (layers "F.Cu" "F.Mask")
+      (net 2 "Net-(J1-Pad2)") (pinfunction "Pin_2") (pintype "passive"))
+    (pad "2" thru_hole oval locked (at 0 2.54 90) (size 1.7 1.7) (drill 1) (layers *.Cu *.Mask)
+      (net 2 "Net-(J1-Pad2)") (pinfunction "Pin_2") (pintype "passive"))
+    (pad "3" thru_hole roundrect locked (at 0 5.08 90) (size 1.7 1.7) (drill 1) (layers *.Cu *.Mask) (roundrect_rratio 0.25)
       (net 5 "GND") (pinfunction "Pin_3") (pintype "passive"))
-    (pad "4" thru_hole oval (at 0 7.62 90) (size 1.7 1.7) (drill 1) (layers *.Cu *.Mask)
+    (pad "3" smd rect locked (at -0.635 5.08 90) (size 1.27 1.7) (layers "F.Cu" "F.Mask")
+      (net 5 "GND") (pinfunction "Pin_3") (pintype "passive"))
+    (pad "3" smd rect locked (at -0.635 5.08 90) (size 1.27 1.7) (layers "B.Cu" "B.Mask")
+      (net 5 "GND") (pinfunction "Pin_3") (pintype "passive"))
+    (pad "4" smd rect locked (at -0.635 7.62 90) (size 1.27 1.7) (layers "F.Cu" "F.Mask")
+      (net 3 "Net-(J1-Pad4)") (pinfunction "Pin_4") (pintype "passive"))
+    (pad "4" thru_hole oval locked (at 0 7.62 90) (size 1.7 1.7) (drill 1) (layers *.Cu *.Mask)
+      (net 3 "Net-(J1-Pad4)") (pinfunction "Pin_4") (pintype "passive"))
+    (pad "4" smd rect locked (at -0.635 7.62 90) (size 1.27 1.7) (layers "B.Cu" "B.Mask")
       (net 3 "Net-(J1-Pad4)") (pinfunction "Pin_4") (pintype "passive"))
     (model "${KICAD6_3DMODEL_DIR}/Connector_PinHeader_2.54mm.3dshapes/PinHeader_1x04_P2.54mm_Vertical.wrl" hide
@@
     (fp_arc (start -1.5 -2.1) (mid -0.75 -2.85) (end 0 -2.1) (layer "B.Mask") (width 0.45))
   )
-  (gr_line (start 157.48 71.12) (end 167.64 71.12) (layer "Edge.Cuts") (width 0.05))
-  (gr_line (start 167.64 58.42) (end 157.48 58.42) (layer "Edge.Cuts") (width 0.05))
-  (gr_line (start 157.48 58.42) (end 157.48 71.12) (layer "Edge.Cuts") (width 0.05))
-  (gr_line (start 167.64 71.12) (end 167.64 58.42) (layer "Edge.Cuts") (width 0.05))
+  (gr_circle (center 158.75 68.58) (end 158.75 68.326) (layer "F.SilkS") (width 0.12) (fill none))
+  (gr_line (start 158.75 68.58) (end 158.75 68.326) (layer "F.SilkS") (width 0.12))
+  (gr_line (start 158.115 71.12) (end 167.005 71.12) (layer "Edge.Cuts") (width 0.05))
+  (gr_arc (start 158.115 71.12) (mid 157.665987 70.934013) (end 157.48 70.485) (layer "Edge.Cuts") (width 0.05))
+  (gr_arc (start 167.64 70.485) (mid 167.454013 70.934013) (end 167.005 71.12) (layer "Edge.Cuts") (width 0.05))
+  (gr_line (start 167.005 58.42) (end 158.115 58.42) (layer "Edge.Cuts") (width 0.05))
+  (gr_line (start 157.48 59.055) (end 157.48 70.485) (layer "Edge.Cuts") (width 0.05))
+  (gr_line (start 167.64 70.485) (end 167.64 59.055) (layer "Edge.Cuts") (width 0.05))
+  (gr_arc (start 167.005 58.42) (mid 167.454013 58.605987) (end 167.64 59.055) (layer "Edge.Cuts") (width 0.05))
+  (gr_arc (start 157.48 59.055) (mid 157.665987 58.605987) (end 158.115 58.42) (layer "Edge.Cuts") (width 0.05))
   (gr_text "SHDN" (at 158.75 68.834 90) (layer "B.SilkS")
     (effects (font (size 1 1) (thickness 0.15)) (justify right mirror))
@@
     (effects (font (size 1 1) (thickness 0.15)) (justify right mirror))
   )
+  (gr_text "↑" (at 161.29 68.58) (layer "F.SilkS")
+    (effects (font (size 0.5 0.5) (thickness 0.1)))
+  )
+  (gr_text "⏚" (at 163.83 68.58) (layer "F.SilkS")
+    (effects (font (size 0.5 0.5) (thickness 0.1)))
+  )
+  (gr_text "www.me.uk" (at 162.814 67.564) (layer "F.SilkS")
+    (effects (font (size 0.5 0.5) (thickness 0.1)))
+  )
+  (gr_text "↓" (at 166.37 68.58) (layer "F.SilkS")
+    (effects (font (size 0.5 0.5) (thickness 0.1)))
+  )
   (segment (start 158.242 64.262) (end 158.626381 64.262) (width 0.25) (layer "F.Cu") (net 1))

Commit message: Tidy up SHDN
Connections:
- J1 pad 2: Net-(J1-Pad2) -> Net-(J1-Pad1)
- U1 pad 2: Net-(J1-Pad2) -> Net-(J1-Pad1)
Routing:
- net Net-(J1-Pad1): track 7.98 -> 17.9 mm
- net Net-(J1-Pad2): track 7.41 -> 0.00 mm

Commit message: Tweak
Parts:
- moved R1 1.02 mm to (166.1, 59.7)
Routing:
- net Net-(R1-Pad2): track 9.35 -> 11.4 mm
Other:
- board text added: "${DATE}"
Changed lines of the file:
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@@
     )
   )
-  (property "DATE" "2022-02-19")
+  (property "DATE" "2022-03-06")
   (net 0 "")
   (net 1 "Net-(J1-Pad1)")
@@
   )
   (footprint "RevK:R_0603" (layer "F.Cu")
-    (at 158.9735 59.679 180)
+    (at 159 59.7 180)
     (descr "Capacitor SMD 0603 (1608 Metric), square (rectangular) end terminal, IPC_7351 nominal, (Body size source: IPC-SM-782 page 76, https://www.pcb-3d.com/wordpress/wp-content/uploads/ipc-sm-782a_amendment_1_and_2.pdf), generated with kicad-footprint-generator")
     (tags "capacitor")
@@
     (pad "2" thru_hole oval locked (at 0 2.54 90) (size 1.7 1.7) (drill 1) (layers *.Cu *.Mask)
       (net 1 "Net-(J1-Pad1)") (pinfunction "Pin_2") (pintype "passive"))
-    (pad "3" thru_hole roundrect locked (at 0 5.08 90) (size 1.7 1.7) (drill 1) (layers *.Cu *.Mask) (roundrect_rratio 0.25)
+    (pad "3" thru_hole roundrect locked (at 0 5.08 90) (size 1.7 1.7) (drill 1) (layers *.Cu *.Mask) (roundrect_rratio 0.1)
       (net 4 "GND") (pinfunction "Pin_3") (pintype "passive"))
     (pad "3" smd rect locked (at -0.635 5.08 90) (size 1.27 1.7) (layers "F.Cu" "F.Mask")
@@
   )
   (footprint "RevK:R_0603" (layer "F.Cu")
-    (at 165.3235 59.044 180)
+    (at 166.1 59.7 180)
     (descr "Capacitor SMD 0603 (1608 Metric), square (rectangular) end terminal, IPC_7351 nominal, (Body size source: IPC-SM-782 page 76, https://www.pcb-3d.com/wordpress/wp-content/uploads/ipc-sm-782a_amendment_1_and_2.pdf), generated with kicad-footprint-generator")
     (tags "capacitor")
@@
   )
   (gr_line (start 157.9 64.9) (end 157.9 68.6) (layer "B.SilkS") (width 0.12))
-  (gr_line (start 159.3 68.58) (end 160.9 68.58) (layer "F.SilkS") (width 0.12))
-  (gr_circle (center 158.75 68.58) (end 158.75 68.326) (layer "F.SilkS") (width 0.12) (fill none))
-  (gr_line (start 158.75 68.58) (end 158.75 68.326) (layer "F.SilkS") (width 0.12))
-  (gr_line (start 160 70.9) (end 160 69.1) (layer "F.Mask") (width 0.5))
+  (gr_circle (center 158.75 68.2) (end 158.75 68.6) (layer "F.SilkS") (width 0.12) (fill none))
+  (gr_line (start 159.5 68.2) (end 160.7 68.2) (layer "F.SilkS") (width 0.12))
+  (gr_line (start 158.75 68.2) (end 158.75 67.8) (layer "F.SilkS") (width 0.12))
+  (gr_line (start 160 70.87) (end 160 69.25) (layer "F.Mask") (width 0.5))
   (gr_line (start 158.115 71.12) (end 167.005 71.12) (layer "Edge.Cuts") (width 0.05))
   (gr_arc (start 158.115 71.12) (mid 157.665987 70.934013) (end 157.48 70.485) (layer "Edge.Cuts") (width 0.05))
@@
     (effects (font (size 1 1) (thickness 0.15)) (justify right mirror))
   )
-  (gr_text "↑" (at 161.29 68.58) (layer "F.SilkS")
+  (gr_text "${DATE}" (at 167.2 62.9 90) (layer "F.SilkS")
     (effects (font (size 0.5 0.5) (thickness 0.1)))
   )
-  (gr_text "⏚" (at 163.83 68.58) (layer "F.SilkS")
+  (gr_text "↑" (at 161.29 68.1) (layer "F.SilkS")
+    (effects (font (size 1 1) (thickness 0.15)))
+  )
+  (gr_text "⏚" (at 163.83 68.1) (layer "F.SilkS")
+    (effects (font (size 1 1) (thickness 0.15)))
+  )
+  (gr_text "www.me.uk" (at 162.5 59.7) (layer "F.SilkS")
     (effects (font (size 0.5 0.5) (thickness 0.1)))
   )
-  (gr_text "www.me.uk" (at 162.814 67.564) (layer "F.SilkS")
-    (effects (font (size 0.5 0.5) (thickness 0.1)))
-  )
-  (gr_text "↓" (at 166.37 68.58) (layer "F.SilkS")
-    (effects (font (size 0.5 0.5) (thickness 0.1)))
+  (gr_text "↓" (at 166.37 68.1) (layer "F.SilkS")
+    (effects (font (size 1 1) (thickness 0.15)))
   )
   (segment (start 158.242 64.262) (end 158.626381 64.262) (width 0.25) (layer "F.Cu") (net 1))
@@
   (segment (start 159.512 68.072) (end 159.22123 68.072) (width 0.5) (layer "F.Cu") (net 1))
   (segment (start 159.7255 64.962) (end 159.066 64.962) (width 0.5) (layer "F.Cu") (net 1))
-  (segment (start 158.75 70) (end 161.29 70) (width 0.25) (layer "F.Cu") (net 1))
+  (segment (start 158.75 70.06) (end 161.29 70.06) (width 0.25) (layer "F.Cu") (net 1))
   (segment (start 159.438007 63.712) (end 159.6255 63.712) (width 0.25) (layer "F.Cu") (net 1))
   (segment (start 157.734 68.834) (end 157.734 64.77) (width 0.25) (layer "F.Cu") (net 1))
@@
   (arc (start 157.734 64.77) (mid 157.88279 64.41079) (end 158.242 64.262) (width 0.25) (layer "F.Cu") (net 1))
   (arc (start 158.75 69.85) (mid 158.03158 69.55242) (end 157.734 68.834) (width 0.25) (layer "F.Cu") (net 1))
-  (segment (start 166.1485 59.044) (end 166.1485 61.994342) (width 0.5) (layer "F.Cu") (net 2))
+  (segment (start 165.9755 60.6495) (end 165.9755 62.412) (width 0.25) (layer "F.Cu") (net 2))
   (segment (start 166.33404 62.412) (end 165.9755 62.412) (width 0.5) (layer "F.Cu") (net 2))
   (segment (start 167.15002 69.06998) (end 167.15002 63.22798) (width 0.5) (layer "F.Cu") (net 2))
   (arc (start 166.1485 61.994342) (mid 166.103539 62.220377) (end 165.9755 62.412) (width 0.5) (layer "F.Cu") (net 2))
   (arc (start 167.15002 63.22798) (mid 166.911025 62.650995) (end 166.33404 62.412) (width 0.5) (layer "F.Cu") (net 2))
+  (arc (start 166.925 59.7) (mid 166.253602 59.978102) (end 165.9755 60.6495) (width 0.25) (layer "F.Cu") (net 2))
   (arc (start 166.37 69.85) (mid 166.921557 69.621537) (end 167.15002 69.06998) (width 0.5) (layer "F.Cu") (net 2))
-  (segment (start 164.4985 59.044) (end 164.33398 58.87948) (width 0.25) (layer "F.Cu") (net 3))
-  (segment (start 159.6255 61.012) (end 158.7825 61.012) (width 0.25) (layer "F.Cu") (net 3))
-  (segment (start 164.33398 58.87948) (end 158.94802 58.87948) (width 0.25) (layer "F.Cu") (net 3))
-  (segment (start 158.1485 59.679) (end 158.1485 60.378) (width 0.25) (layer "F.Cu") (net 3))
-  (arc (start 158.7825 61.012) (mid 158.334194 60.826306) (end 158.1485 60.378) (width 0.25) (layer "F.Cu") (net 3))
-  (arc (start 158.94802 58.87948) (mid 158.382674 59.113654) (end 158.1485 59.679) (width 0.25) (layer "F.Cu") (net 3))
+  (segment (start 164.33398 58.87948) (end 163.07948 58.87948) (width 0.25) (layer "F.Cu") (net 3))
+  (segment (start 159.487 61.012) (end 159.6255 61.012) (width 0.25) (layer "F.Cu") (net 3))
+  (segment (start 163.07948 58.87948) (end 158.99552 58.87948) (width 0.25) (layer "F.Cu") (net 3))
+  (segment (start 163.07948 58.87948) (end 164.45448 58.87948) (width 0.25) (layer "F.Cu") (net 3))
+  (arc (start 158.175 59.7) (mid 158.559276 60.627724) (end 159.487 61.012) (width 0.25) (layer "F.Cu") (net 3))
+  (arc (start 164.45448 58.87948) (mid 165.034675 59.119805) (end 165.275 59.7) (width 0.25) (layer "F.Cu") (net 3))
+  (arc (start 158.99552 58.87948) (mid 158.415325 59.119805) (end 158.175 59.7) (width 0.25) (layer "F.Cu") (net 3))
   (segment (start 162.8545 65.532) (end 164.338 65.532) (width 0.5) (layer "F.Cu") (net 4))
-  (segment (start 159.7985 59.679) (end 160.5755 60.456) (width 0.25) (layer "F.Cu") (net 4))
-  (segment (start 160.5755 60.456) (end 160.5755 61.012) (width 0.25) (layer "F.Cu") (net 4))
+  (segment (start 160.5755 61.012) (end 160.5755 60.4505) (width 0.25) (layer "F.Cu") (net 4))
   (via (at 162.8545 65.532) (size 1) (drill 0.5) (layers "F.Cu" "B.Cu") (net 4))
+  (arc (start 160.5755 60.4505) (mid 160.355684 59.919816) (end 159.825 59.7) (width 0.25) (layer "F.Cu") (net 4))
   (zone (net 4) (net_name "GND") (layers F&B.Cu) (hatch edge 0.508)
     (connect_pads (clearance 0.254))

Commit message: Tweak
Routing:
- net Net-(R1-Pad2): track 11.4 -> 10.1 mm
Changed lines of the file:
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@@
   (segment (start 166.33404 62.412) (end 165.9755 62.412) (width 0.5) (layer "F.Cu") (net 2))
   (segment (start 167.15002 69.06998) (end 167.15002 63.22798) (width 0.5) (layer "F.Cu") (net 2))
-  (arc (start 166.1485 61.994342) (mid 166.103539 62.220377) (end 165.9755 62.412) (width 0.5) (layer "F.Cu") (net 2))
   (arc (start 167.15002 63.22798) (mid 166.911025 62.650995) (end 166.33404 62.412) (width 0.5) (layer "F.Cu") (net 2))
   (arc (start 166.925 59.7) (mid 166.253602 59.978102) (end 165.9755 60.6495) (width 0.25) (layer "F.Cu") (net 2))
   (arc (start 166.37 69.85) (mid 166.921557 69.621537) (end 167.15002 69.06998) (width 0.5) (layer "F.Cu") (net 2))
-  (segment (start 164.33398 58.87948) (end 163.07948 58.87948) (width 0.25) (layer "F.Cu") (net 3))
   (segment (start 159.487 61.012) (end 159.6255 61.012) (width 0.25) (layer "F.Cu") (net 3))
-  (segment (start 163.07948 58.87948) (end 158.99552 58.87948) (width 0.25) (layer "F.Cu") (net 3))
-  (segment (start 163.07948 58.87948) (end 164.45448 58.87948) (width 0.25) (layer "F.Cu") (net 3))
+  (segment (start 158.99552 58.87948) (end 164.45448 58.87948) (width 0.25) (layer "F.Cu") (net 3))
   (arc (start 158.175 59.7) (mid 158.559276 60.627724) (end 159.487 61.012) (width 0.25) (layer "F.Cu") (net 3))
   (arc (start 164.45448 58.87948) (mid 165.034675 59.119805) (end 165.275 59.7) (width 0.25) (layer "F.Cu") (net 3))

Commit message: Tweaks
Other:
- rule pad_to_mask_clearance: 0 -> 0.125
Changed lines of the file:
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@@
       (dielectric_constraints no)
     )
-    (pad_to_mask_clearance 0)
+    (pad_to_mask_clearance 0.125)
     (pad_to_paste_clearance_ratio -0.02)
     (pcbplotparams
@@
     (effects (font (size 1 1) (thickness 0.15)))
   )
-  (segment (start 158.242 64.262) (end 158.626381 64.262) (width 0.25) (layer "F.Cu") (net 1))
   (segment (start 158.55098 67.40175) (end 158.55098 65.47702) (width 0.5) (layer "F.Cu") (net 1))
   (segment (start 159.512 68.072) (end 159.22123 68.072) (width 0.5) (layer "F.Cu") (net 1))
   (segment (start 159.7255 64.962) (end 159.066 64.962) (width 0.5) (layer "F.Cu") (net 1))
   (segment (start 158.75 70.06) (end 161.29 70.06) (width 0.25) (layer "F.Cu") (net 1))
-  (segment (start 159.438007 63.712) (end 159.6255 63.712) (width 0.25) (layer "F.Cu") (net 1))
-  (segment (start 157.734 68.834) (end 157.734 64.77) (width 0.25) (layer "F.Cu") (net 1))
-  (segment (start 159.073003 64.077003) (end 159.438007 63.712) (width 0.25) (layer "F.Cu") (net 1))
-  (arc (start 158.626381 64.262) (mid 158.868091 64.21392) (end 159.073003 64.077003) (width 0.25) (layer "F.Cu") (net 1))
+  (segment (start 158 64.888381) (end 158 69.1) (width 0.25) (layer "F.Cu") (net 1))
+  (segment (start 159.6255 63.712) (end 159.438007 63.712) (width 0.25) (layer "F.Cu") (net 1))
+  (segment (start 159.438007 63.712) (end 159.073003 64.077003) (width 0.25) (layer "F.Cu") (net 1))
   (arc (start 159.22123 68.072) (mid 158.747292 67.875688) (end 158.55098 67.40175) (width 0.5) (layer "F.Cu") (net 1))
+  (arc (start 159.073003 64.077003) (mid 158.868091 64.21392) (end 158.626381 64.262) (width 0.25) (layer "F.Cu") (net 1))
   (arc (start 161.29 69.85) (mid 160.769236 68.592764) (end 159.512 68.072) (width 0.5) (layer "F.Cu") (net 1))
   (arc (start 159.066 64.962) (mid 158.701826 65.112846) (end 158.55098 65.47702) (width 0.5) (layer "F.Cu") (net 1))
-  (arc (start 157.734 64.77) (mid 157.88279 64.41079) (end 158.242 64.262) (width 0.25) (layer "F.Cu") (net 1))
-  (arc (start 158.75 69.85) (mid 158.03158 69.55242) (end 157.734 68.834) (width 0.25) (layer "F.Cu") (net 1))
+  (arc (start 158 69.1) (mid 158.21967 69.63033) (end 158.75 69.85) (width 0.25) (layer "F.Cu") (net 1))
+  (arc (start 158.626381 64.262) (mid 158.183463 64.445463) (end 158 64.888381) (width 0.25) (layer "F.Cu") (net 1))
   (segment (start 165.9755 60.6495) (end 165.9755 62.412) (width 0.25) (layer "F.Cu") (net 2))
   (segment (start 166.33404 62.412) (end 165.9755 62.412) (width 0.5) (layer "F.Cu") (net 2))

Commit message: Revised rules
Other:
- rule pad_to_mask_clearance: 0.125 -> 0.01
