File: Regulator/Regulator.kicad_pcb (KiCad board)
At the start: 2 copper layers, 10.2 x 12.7 mm, 10 parts, among them J1 Conn_01x04, U1 LMR16006+FB

Commit message: Tidy regulator
Parts:
- C1: value 0.1uF -> 100nF; footprint RevK:Hidden -> RevK:C_0603_
- C2, C3: footprint RevK:Hidden -> RevK:C_0805_
- D1: footprint RevK:Hidden -> RevK:D_1206_
- L1: footprint RevK:Hidden -> RevK:L_4x4_
- turned D1 to 0 degrees
- turned L1 to 0 degrees

Commit message: Tidy
Parts:
- U1: footprint RevK:RegulatorBlockFB -> RevK:SOT-23-Thin-6-Reg

Commit message: New production files
Parts:
- U1: value LMR16006+FB -> LMR16006XDDCR
Other:
- rule pad_to_mask_clearance: 0.01 -> 0
Changed lines of the file:
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@@
       (dielectric_constraints no)
     )
-    (pad_to_mask_clearance 0.01)
+    (pad_to_mask_clearance 0)
     (pad_to_paste_clearance_ratio -0.02)
     (pcbplotparams
@@
     (at 160.5755 62.362)
     (descr "LMR16006 based fixed regulator")
-    (property "Manufacturer" "TI")
-    (property "Part No" "LMR16006YQ3")
+    (property "LCSC Part" "C87080")
     (property "Sheetfile" "Regulator.kicad_sch")
     (property "Sheetname" "")
@@
       (effects (font (size 0.5 0.5) (thickness 0.08)))
     )
-    (fp_text value "LMR16006+FB" (at -2.65 -2.55 180) (layer "F.Fab")
+    (fp_text value "LMR16006XDDCR" (at -2.65 -2.55 180) (layer "F.Fab")
       (effects (font (size 0.5 0.5) (thickness 0.1)) (justify left))
     )

Commit message: Working on assembly files
Parts:
- J1: footprint Connector_PinHeader_2.54mm:PinHeader_1x04_P2.54mm_Vertical -> RevK:PinHeader_1x04_P2.54mm_Right
- L1: footprint RevK:L_4x4_ -> RevK:L_1210_
- R1: value 10M 1% or 0R -> 10M 1%
- R2: value 1.8M 1% or NF -> 1.8M 1%
- U1: footprint RevK:SOT-23-Thin-6-Reg -> RevK:SOT-23-Thin-6-Reg2
- moved J1 3.81 mm to (162.6, 69.8), turned to 0 degrees
- turned U1 to -90 degrees
Routing:
- net Net-(R1-Pad1): track 11.9 -> 9.44 mm
