File: LMR16006/Regulator.kicad_sch (KiCad schematic)
At the start: 10 parts, among them J1 Conn_01x04, U1 LMR16006XDDCR

Commit message: Put back regulator
Parts:
- J1: footprint RevK:PinHeader_1x04_P2.54mm_Right -> RevK:JLC-PinHeader_1x04_P2.54mm_Right
- L1: footprint RevK:L_1210_ -> RevK:L_4x4_; LCSC Part # C560045 -> C354575
- U1: footprint RevK:SOT-23-Thin-6-Reg2 -> RevK:SOT-23-Thin-6-Reg
Changed lines of the file:
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@@
       (effects (font (size 1.27 1.27)) (justify right))
     )
-    (property "Footprint" "RevK:L_1210_" (id 2) (at 116.84 60.96 0)
+    (property "Footprint" "RevK:L_4x4_" (id 2) (at 116.84 60.96 0)
       (effects (font (size 1.27 1.27)) hide)
     )
@@
       (effects (font (size 1.27 1.27)) hide)
     )
-    (property "LCSC Part #" "C560045" (id 6) (at 116.84 60.96 0)
+    (property "LCSC Part #" "C354575" (id 6) (at 116.84 60.96 0)
       (effects (font (size 1.27 1.27)) hide)
     )
@@
     (property "Reference" "J1" (id 0) (at 84.455 50.2752 0))
     (property "Value" "Conn_01x04" (id 1) (at 84.455 52.8121 0))
-    (property "Footprint" "RevK:PinHeader_1x04_P2.54mm_Right" (id 2) (at 84.455 57.785 0)
+    (property "Footprint" "RevK:JLC-PinHeader_1x04_P2.54mm_Right" (id 2) (at 84.455 57.785 0)
       (effects (font (size 1.27 1.27)) hide)
     )
@@
       (effects (font (size 1.27 1.27)) (justify left))
     )
-    (property "Footprint" "RevK:SOT-23-Thin-6-Reg2" (id 2) (at 112.395 52.705 0)
+    (property "Footprint" "RevK:SOT-23-Thin-6-Reg" (id 2) (at 112.395 52.705 0)
       (effects (font (size 1.27 1.27)) hide)
     )
@@
     )
     (path "/a5323771-5ccb-4d0d-b118-cd57dcc7b6cd"
-      (reference "J1") (unit 1) (value "Conn_01x04") (footprint "RevK:PinHeader_1x04_P2.54mm_Right")
+      (reference "J1") (unit 1) (value "Conn_01x04") (footprint "RevK:JLC-PinHeader_1x04_P2.54mm_Right")
     )
     (path "/00000000-0000-0000-0000-0000610fe01a"
-      (reference "L1") (unit 1) (value "6.8uH") (footprint "RevK:L_1210_")
+      (reference "L1") (unit 1) (value "6.8uH") (footprint "RevK:L_4x4_")
     )
     (path "/ab097fcc-5168-4497-a352-43eecc18a0c7"
@@
     )
     (path "/aff7249d-1a70-46a9-947a-070a2f7d9e4a"
-      (reference "U1") (unit 1) (value "LMR16006XDDCR") (footprint "RevK:SOT-23-Thin-6-Reg2")
+      (reference "U1") (unit 1) (value "LMR16006XDDCR") (footprint "RevK:SOT-23-Thin-6-Reg")
     )
   )

Commit message: Tweaks for production
Parts:
- removed U1: LMR16006XDDCR, RevK:SOT-23-Thin-6-Reg, symbol RevK:LMR16006+FB
- added U1: LMR16006XDDCR, RevK:SOT-23-Thin-6-Reg, symbol RevK:LMR16006XDDCR
- C2, C3: Note 0603 or 0805 -> (none)
Connections:
- net GND: now also U1.2 (GND)
- net at J1.4 (Pin_4), R1.1: now also U1.7 (VOUT)
- net at R1.2, R2.2: now also U1.3 (FB)
- net at J1.1 (Pin_1), J1.2 (Pin_2): now also U1.4 (SHDN), U1.5 (VIN)
Changed lines of the file:
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@@
-      (effects (font (size 1.27 1.27)) hide)
-    )
-    (property "Note" "0603 or 0805" (id 4) (at 116.84 57.15 0)
       (effects (font (size 1.27 1.27)) hide)
     )
@@
       (effects (font (size 1.27 1.27)) hide)
     )
-    (property "Note" "0603 or 0805" (id 4) (at 116.84 59.055 0)
-      (effects (font (size 1.27 1.27)) hide)
-    )
     (property "LCSC Part #" "C17024" (id 5) (at 116.84 59.055 0)
       (effects (font (size 1.27 1.27)) hide)
@@
     (pin "1")
     (pin "2")
+  )
+  (symbol (lib_id "RevK:LMR16006XDDCR") (at 100.965 55.245 0) (unit 1)
+    (in_bom yes) (on_board yes) (fields_autoplaced)
+    (property "Reference" "U1" (id 0) (at 118.745 50.4022 0))
+    (property "Value" "LMR16006XDDCR" (id 1) (at 118.745 52.9391 0))
+    (property "Footprint" "RevK:SOT-23-Thin-6-Reg" (id 2) (at 116.205 71.755 0)
+      (effects (font (size 1.27 1.27)) hide)
+    )
+    (property "Datasheet" "" (id 3) (at 112.395 52.705 0)
+      (effects (font (size 1.27 1.27)) hide)
+    )
+    (property "Manufacturer" "TI" (id 4) (at 128.905 69.85 0)
+      (effects (font (size 1.27 1.27)) hide)
+    )
+    (property "Part No" "LMR16006XDDCR" (id 5) (at 119.38 69.85 0)
+      (effects (font (size 1.27 1.27)) hide)
+    )
+    (property "LCSC Part #" "C87080" (id 6) (at 106.68 69.85 0)
+      (effects (font (size 1.27 1.27)) hide)
+    )
+    (property "JLCPCB Rotation Offset" "90" (id 7) (at 131.445 69.85 0)
+      (effects (font (size 1.27 1.27)) hide)
+    )
+    (pin "1")
+    (pin "2")
+    (pin "3")
+    (pin "4")
+    (pin "5")
+    (pin "6")
+    (pin "7")
   )
   (symbol (lib_id "Connector_Generic:Conn_01x04") (at 84.455 57.785 0) (mirror y) (unit 1)
@@
     )
   )
-  (symbol (lib_id "RevK:LMR16006+FB") (at 100.965 55.245 0) (unit 1)
-    (in_bom yes) (on_board yes) (fields_autoplaced)
-    (property "Reference" "U1" (id 0) (at 134.62 59.4903 0)
-      (effects (font (size 1.27 1.27)) (justify left))
-    )
-    (property "Value" "LMR16006XDDCR" (id 1) (at 134.62 62.0272 0)
-      (effects (font (size 1.27 1.27)) (justify left))
-    )
-    (property "Footprint" "RevK:SOT-23-Thin-6-Reg" (id 2) (at 112.395 52.705 0)
-      (effects (font (size 1.27 1.27)) hide)
-    )
-    (property "Datasheet" "~" (id 3) (at 112.395 52.705 0)
-      (effects (font (size 1.27 1.27)) hide)
-    )
-    (property "LCSC Part #" "C87080" (id 4) (at 100.965 55.245 0)
-      (effects (font (size 1.27 1.27)) hide)
-    )
-    (pin "1")
-    (pin "2")
-    (pin "3")
-    (pin "4")
-    (pin "5")
-  )
   (symbol (lib_id "Device:R") (at 97.155 68.58 90) (unit 1)
     (in_bom yes) (on_board yes)
@@
       (reference "R2") (unit 1) (value "30k 1%") (footprint "RevK:R_0603")
     )
-    (path "/aff7249d-1a70-46a9-947a-070a2f7d9e4a"
+    (path "/6d25a0f6-ef0a-4401-a1d1-0fee69fa15d1"
       (reference "U1") (unit 1) (value "LMR16006XDDCR") (footprint "RevK:SOT-23-Thin-6-Reg")
     )
