File: PCB/Reference/Reference.kicad_sch (KiCad schematic)
At the start: 10 parts, among them J1 Conn_01x04, U1 LMR16006XDDCR

Commit message: Add new reg, and tidy
Parts:
- added C4: 10uF 50V, RevK:C_0603_, symbol RevK:Hidden
- added C5: 10uF 6.3V, RevK:C_0603_, symbol RevK:Hidden
- added C6: 100nF, RevK:C_0603_, symbol RevK:Hidden
- added L2: 10uH, RevK:L_4x4_, symbol RevK:Hidden
- added R3: 124k, RevK:R_0402_, symbol RevK:Hidden
- added R4: 40k2, RevK:R_0402_, symbol RevK:Hidden
- added R5: 1M, RevK:R_0402_, symbol RevK:Hidden
- added U2: MD8942, RevK:SOT-23-6-MD8942, symbol RevK:MD89420-RegBlock
Connections:
- net GND: now also U2.2 (GND), U2.7 (GND)
- new net +3.3V: U2.8 (VOUT)
- new net DC: U2.5 (VIN)
- no-connect marks 0 -> 1
