File: PCB/Reference/Reference.kicad_sch (KiCad schematic)
At the start: 18 parts, among them J1 Conn_01x04, U1 LMR16006XDDCR, U2 MD8942

Commit message: Tidy
Parts:
- added D1: RGB, RevK:LED-RGB-1.6x1.6, symbol Device:LED_RBGA
- added FID1, FID2, FID3, FID4, FID5, FID6, FID7, FID8: Fiducial, Fiducial:Fiducial_1mm_Mask2mm, symbol Mechanical:Fiducial
- added H1, H2, H3, H4: MountingHole, MountingHole:MountingHole_2mm, symbol Mechanical:MountingHole
- added R1: 680R, RevK:R_0402, symbol Device:R
- added R2: 2K, RevK:R_0402, symbol Device:R
- added R3: 220R, RevK:R_0402, symbol Device:R
- added U2, U6: Barcode, RevK:EAN-5060634238069, symbol RevK:Barcode
Connections:
- net +3.3V: now also D1.4 (A)
- new net: D1.3 (GK), R2.1
- new net: D1.1 (RK), R1.1
- new net: D1.2 (BK), R3.1
- new net B: R3.2
- new net G: R2.2
- new net R: R1.2

Commit message: Tidy
Parts:
- removed H1, H2, H3, H4: MountingHole, MountingHole:MountingHole_2mm, symbol Mechanical:MountingHole
- removed U6: Barcode, RevK:EAN-5060634238069, symbol RevK:Barcode
Other:
- moved on the sheet: FID1, FID2, FID3, FID4, FID5, FID6, FID7, FID8

Commit message: PCB templatge
Parts:
- removed FID1, FID2, FID3, FID4, FID5, FID6, FID7, FID8: Fiducial, Fiducial:Fiducial_1mm_Mask2mm, symbol Mechanical:Fiducial
- added C7: 0.1uF, RevK:C_0402, symbol Device:C
- added PCB1: 70x70, RevK:PCB7070, symbol RevK:PCB
- added R9: 4k7, RevK:R_0402, symbol Device:R
- added U4: CH340X, RevK:CH340X, symbol RevK:CH340X
Connections:
- net +3.3V: now also C7.1, R9.1, U4.10 (V3), U4.7 (VCC)
- net GND: now also C7.2, U4.3 (GND), U4.5 (~{CTS})
- new net BOOT: R9.2, U4.6 (TNOW/~{DTR})
- new net D+: U4.1 (UD+)
- new net D-: U4.2 (UD-)
- new net EN: U4.4 (~{RTS})
- new net I: U4.8 (TXD)
- new net O: U4.9 (RXD)
Other:
- moved on the sheet: C1, C2, C3, D1, J1, L1, R1, R2, R3, U1

Commit message: Tweak
Parts:
- U4: JLCPCB Rotation Offset 90 -> -90
Connections:
- net +3.3V: no longer R9.1
- net GND: no longer U4.5 (~{CTS})
- new net: R9.1, U4.5 (~{CTS})
Other:
- moved on the sheet: R9
Changed lines of the file:
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@@
   (junction (at 93.345 52.07) (diameter 0) (color 0 0 0 0)
   )
+  (junction (at 120.015 160.02) (diameter 0) (color 0 0 0 0)
+  )
   (junction (at 107.95 138.43) (diameter 0) (color 0 0 0 0)
   )
@@
   )
   (junction (at 97.155 57.15) (diameter 0) (color 0 0 0 0)
-  )
-  (junction (at 127.635 160.02) (diameter 0) (color 0 0 0 0)
   )
   (junction (at 94.615 62.865) (diameter 0) (color 0 0 0 0)
@@
     (stroke (width 0) (type default))
   )
-  (wire (pts (xy 127.635 157.48) (xy 127.635 160.02))
-    (stroke (width 0) (type default))
-  )
   (wire (pts (xy 97.155 62.865) (xy 94.615 62.865))
     (stroke (width 0) (type default))
   )
-  (wire (pts (xy 127.635 160.02) (xy 128.905 160.02))
-    (stroke (width 0) (type default))
-  )
   (wire (pts (xy 106.68 138.43) (xy 107.95 138.43))
     (stroke (width 0) (type default))
@@
     (stroke (width 0) (type default))
   )
-  (wire (pts (xy 118.11 160.02) (xy 127.635 160.02))
+  (wire (pts (xy 122.555 160.02) (xy 120.015 160.02))
+    (stroke (width 0) (type default))
+  )
+  (wire (pts (xy 120.015 152.4) (xy 118.11 152.4))
     (stroke (width 0) (type default))
   )
   (wire (pts (xy 97.155 57.15) (xy 104.775 57.15))
+    (stroke (width 0) (type default))
+  )
+  (wire (pts (xy 120.015 160.02) (xy 118.11 160.02))
     (stroke (width 0) (type default))
   )
@@
     )
   )
-  (global_label "BOOT" (shape output) (at 128.905 160.02 0) (fields_autoplaced)
+  (global_label "BOOT" (shape output) (at 122.555 160.02 0) (fields_autoplaced)
     (effects (font (size 1.27 1.27)) (justify left))
-    (property "Intersheetrefs" "${INTERSHEET_REFS}" (at 136.0552 160.02 0)
+    (property "Intersheetrefs" "${INTERSHEET_REFS}" (at 129.7052 160.02 0)
       (effects (font (size 1.27 1.27)) (justify left) hide)
     )
@@
     )
   )
-  (symbol (lib_id "power:+3.3V") (at 127.635 149.86 0) (unit 1)
-    (in_bom yes) (on_board yes) (dnp no) (fields_autoplaced)
-    (property "Reference" "#PWR010" (at 127.635 153.67 0)
-      (effects (font (size 1.27 1.27)) hide)
-    )
-    (property "Value" "+3.3V" (at 127.635 146.2842 0)
-      (effects (font (size 1.27 1.27)))
-    )
-    (property "Footprint" "" (at 127.635 149.86 0)
-      (effects (font (size 1.27 1.27)) hide)
-    )
-    (property "Datasheet" "" (at 127.635 149.86 0)
-      (effects (font (size 1.27 1.27)) hide)
-    )
-    (pin "1")
-    (instances
-      (project "Reference"
-        (path "/825c70b0-4860-42b7-97dc-86bfa46e06fd"
-          (reference "#PWR010") (unit 1)
-        )
-      )
-      (project "Generic"
-        (path "/babeabf2-f3b0-4ed5-8d9e-0215947e6cf3"
-          (reference "#PWR07") (unit 1)
-        )
-      )
-    )
-  )
   (symbol (lib_id "RevK:Hidden") (at 118.745 99.06 270) (unit 1)
     (in_bom yes) (on_board yes) (dnp no)
@@
         (path "/babeabf2-f3b0-4ed5-8d9e-0215947e6cf3"
           (reference "R12") (unit 1)
-        )
-      )
-    )
-  )
-  (symbol (lib_id "power:GND") (at 118.11 156.21 90) (unit 1)
-    (in_bom yes) (on_board yes) (dnp no)
-    (property "Reference" "#PWR09" (at 124.46 156.21 0)
-      (effects (font (size 1.27 1.27)) hide)
-    )
-    (property "Value" "GND" (at 121.3612 156.083 90)
-      (effects (font (size 1.27 1.27)) (justify right))
-    )
-    (property "Footprint" "" (at 118.11 156.21 0)
-      (effects (font (size 1.27 1.27)) hide)
-    )
-    (property "Datasheet" "" (at 118.11 156.21 0)
-      (effects (font (size 1.27 1.27)) hide)
-    )
-    (pin "1")
-    (instances
-      (project "Reference"
-        (path "/825c70b0-4860-42b7-97dc-86bfa46e06fd"
-          (reference "#PWR09") (unit 1)
-        )
-      )
-      (project "Generic"
-        (path "/babeabf2-f3b0-4ed5-8d9e-0215947e6cf3"
-          (reference "#PWR012") (unit 1)
         )
       )
@@
       (effects (font (size 1.27 1.27)) hide)
     )
-    (property "JLCPCB Rotation Offset" "90" (at 107.95 153.67 0)
+    (property "JLCPCB Rotation Offset" "-90" (at 107.95 153.67 0)
       (effects (font (size 1.27 1.27)) hide)
     )
@@
     )
   )
-  (symbol (lib_id "Device:R") (at 127.635 153.67 0) (unit 1)
-    (in_bom yes) (on_board yes) (dnp no)
-    (property "Reference" "R9" (at 129.54 153.67 90)
-      (effects (font (size 1.27 1.27)))
-    )
-    (property "Value" "4k7" (at 127.635 153.67 90)
-      (effects (font (size 1.27 1.27)))
-    )
-    (property "Footprint" "RevK:R_0402" (at 125.857 153.67 90)
-      (effects (font (size 1.27 1.27)) hide)
-    )
-    (property "Datasheet" "~" (at 127.635 153.67 0)
-      (effects (font (size 1.27 1.27)) hide)
-    )
+  (symbol (lib_id "Device:R") (at 120.015 156.21 0) (unit 1)
+    (in_bom yes) (on_board yes) (dnp no)
+    (property "Reference" "R9" (at 121.92 156.21 90)
+      (effects (font (size 1.27 1.27)))
+    )
+    (property "Value" "4k7" (at 120.015 156.21 90)
+      (effects (font (size 1.27 1.27)))
+    )
+    (property "Footprint" "RevK:R_0402" (at 118.237 156.21 90)
+      (effects (font (size 1.27 1.27)) hide)
+    )
+    (property "Datasheet" "~" (at 120.015 156.21 0)
+      (effects (font (size 1.27 1.27)) hide)
+    )

Commit message: VCut
Parts:
- added V1, V2: ~, RevK:VCUT70, symbol RevK:VCUT
Changed lines of the file:
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@@
+    )
+  )
+  (symbol (lib_id "RevK:VCUT") (at 245.11 177.165 180) (unit 1)
+    (in_bom yes) (on_board yes) (dnp no) (fields_autoplaced)
+    (property "Reference" "V2" (at 245.11 178.435 0)
+      (effects (font (size 1.27 1.27)) hide)
+    )
+    (property "Value" "~" (at 245.11 177.165 0)
+      (effects (font (size 1.27 1.27)))
+    )
+    (property "Footprint" "RevK:VCUT70" (at 245.11 175.895 0)
+      (effects (font (size 1.27 1.27)) hide)
+    )
+    (property "Datasheet" "" (at 245.11 177.165 0)
+      (effects (font (size 1.27 1.27)) hide)
+    )
+    (instances
+      (project "Reference"
+        (path "/825c70b0-4860-42b7-97dc-86bfa46e06fd"
+          (reference "V2") (unit 1)
+        )
+      )
     )
   )
@@
         )
       )
+    )
+  )
+  (symbol (lib_id "RevK:VCUT") (at 245.11 170.815 0) (unit 1)
+    (in_bom yes) (on_board yes) (dnp no) (fields_autoplaced)
+    (property "Reference" "V1" (at 245.11 169.545 0)
+      (effects (font (size 1.27 1.27)) hide)
+    )
+    (property "Value" "~" (at 245.11 170.815 0)
+      (effects (font (size 1.27 1.27)))
+    )
+    (property "Footprint" "RevK:VCUT70" (at 245.11 172.085 0)
+      (effects (font (size 1.27 1.27)) hide)
+    )
+    (property "Datasheet" "" (at 245.11 170.815 0)
+      (effects (font (size 1.27 1.27)) hide)
+    )
+    (instances
+      (project "Reference"
+        (path "/825c70b0-4860-42b7-97dc-86bfa46e06fd"
+          (reference "V1") (unit 1)
+        )
+      )

Commit message: CH340X DTR
Parts:
- removed R9: 4k7, RevK:R_0402, symbol Device:R
- V1, V2: now left out of the parts list
Connections:
- net BOOT: now also U4.5 (~{CTS})
Changed lines of the file:
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@@
   (junction (at 93.345 52.07) (diameter 0) (color 0 0 0 0)
   )
-  (junction (at 120.015 160.02) (diameter 0) (color 0 0 0 0)
-  )
   (junction (at 107.95 138.43) (diameter 0) (color 0 0 0 0)
   )
   (junction (at 93.345 49.53) (diameter 0) (color 0 0 0 0)
+  )
+  (junction (at 118.11 160.02) (diameter 0) (color 0 0 0 0)
   )
   (junction (at 97.155 57.15) (diameter 0) (color 0 0 0 0)
@@
     (stroke (width 0) (type default))
   )
+  (wire (pts (xy 118.11 152.4) (xy 118.11 160.02))
+    (stroke (width 0) (type default))
+  )
   (wire (pts (xy 97.155 62.865) (xy 94.615 62.865))
     (stroke (width 0) (type default))
@@
     (stroke (width 0) (type default))
   )
-  (wire (pts (xy 122.555 160.02) (xy 120.015 160.02))
-    (stroke (width 0) (type default))
-  )
-  (wire (pts (xy 120.015 152.4) (xy 118.11 152.4))
+  (wire (pts (xy 118.11 160.02) (xy 119.38 160.02))
     (stroke (width 0) (type default))
   )
   (wire (pts (xy 97.155 57.15) (xy 104.775 57.15))
-    (stroke (width 0) (type default))
-  )
-  (wire (pts (xy 120.015 160.02) (xy 118.11 160.02))
     (stroke (width 0) (type default))
   )
@@
     )
   )
-  (global_label "BOOT" (shape output) (at 122.555 160.02 0) (fields_autoplaced)
+  (global_label "BOOT" (shape output) (at 119.38 160.02 0) (fields_autoplaced)
     (effects (font (size 1.27 1.27)) (justify left))
-    (property "Intersheetrefs" "${INTERSHEET_REFS}" (at 129.7052 160.02 0)
+    (property "Intersheetrefs" "${INTERSHEET_REFS}" (at 126.5302 160.02 0)
       (effects (font (size 1.27 1.27)) (justify left) hide)
     )
@@
   )
   (symbol (lib_id "RevK:VCUT") (at 245.11 177.165 180) (unit 1)
-    (in_bom yes) (on_board yes) (dnp no) (fields_autoplaced)
+    (in_bom no) (on_board yes) (dnp no) (fields_autoplaced)
     (property "Reference" "V2" (at 245.11 178.435 0)
       (effects (font (size 1.27 1.27)) hide)
@@
     )
     (property "Datasheet" "" (at 245.11 177.165 0)
+      (effects (font (size 1.27 1.27)) hide)
+    )
+    (property "Sim.Enable" "0" (at 245.11 177.165 0)
       (effects (font (size 1.27 1.27)) hide)
     )
@@
     )
   )
-  (symbol (lib_id "Device:R") (at 120.015 156.21 0) (unit 1)
-    (in_bom yes) (on_board yes) (dnp no)
-    (property "Reference" "R9" (at 121.92 156.21 90)
-      (effects (font (size 1.27 1.27)))
-    )
-    (property "Value" "4k7" (at 120.015 156.21 90)
-      (effects (font (size 1.27 1.27)))
-    )
-    (property "Footprint" "RevK:R_0402" (at 118.237 156.21 90)
-      (effects (font (size 1.27 1.27)) hide)
-    )
-    (property "Datasheet" "~" (at 120.015 156.21 0)
-      (effects (font (size 1.27 1.27)) hide)
-    )
-    (pin "1")
-    (pin "2")
-    (instances
-      (project "Reference"
-        (path "/825c70b0-4860-42b7-97dc-86bfa46e06fd"
-          (reference "R9") (unit 1)
-        )
-      )
-      (project "Generic"
-        (path "/babeabf2-f3b0-4ed5-8d9e-0215947e6cf3"
-          (reference "R6") (unit 1)
-        )
-      )
-    )
-  )
   (symbol (lib_id "Device:R") (at 100.965 62.865 90) (unit 1)
     (in_bom yes) (on_board yes) (dnp no)
@@
   )
   (symbol (lib_id "RevK:VCUT") (at 245.11 170.815 0) (unit 1)
-    (in_bom yes) (on_board yes) (dnp no) (fields_autoplaced)
+    (in_bom no) (on_board yes) (dnp no) (fields_autoplaced)
     (property "Reference" "V1" (at 245.11 169.545 0)
       (effects (font (size 1.27 1.27)) hide)
@@
       (effects (font (size 1.27 1.27)) hide)
     )
+    (property "Sim.Enable" "0" (at 245.11 170.815 0)
+      (effects (font (size 1.27 1.27)) hide)
+    )

Commit message: Fix RGB and tidy
Parts:
- D1: symbol Device:LED_RBGA -> Device:LED_RGBA
Connections:
- net at R2.1: now also D1.2 (GK); no longer D1.3 (GK)
- net at R3.1: now also D1.3 (BK); no longer D1.2 (BK)
Changed lines of the file:
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@@
     )
   )
-  (symbol (lib_id "Device:LED_RBGA") (at 176.53 60.96 0) (unit 1)
+  (symbol (lib_id "Device:LED_RGBA") (at 176.53 60.96 0) (unit 1)
     (in_bom yes) (on_board yes) (dnp no)
     (property "Reference" "D1" (at 176.53 48.3362 0)
