File: PCB/Reference/Reference.kicad_sch (KiCad schematic)
At the start: 28 parts, among them J1 Conn_01x04, U1 LMR16006XDDCR, U2 Barcode, U2 MD8942, U4 CH340X

Commit message: dot
Parts:
- R4: value 40k2 -> 39k2
Changed lines of the file:
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@@
       (effects (font (size 1.27 1.27)))
     )
-    (property "Value" "40k2" (at 125.095 99.06 90)
+    (property "Value" "39k2" (at 125.095 99.06 90)
       (effects (font (size 1.27 1.27)) (justify left))
     )

Commit message: Tidy
Parts:
- removed C1: 100nF, RevK:C_0603_, symbol RevK:Hidden
- removed C2: 2.2uF, RevK:C_0805_, symbol RevK:Hidden
- removed C3: 10uF, RevK:C_0805_, symbol RevK:Hidden
- removed D1: Schottky, RevK:D_1206_, symbol RevK:Hidden
- removed J1: Conn_01x04, RevK:JLC-PinHeader_1x04_P2.54mm_Right, symbol Connector_Generic:Conn_01x04
- removed L1: 6.8uH, RevK:L_4x4_, symbol RevK:Hidden
- removed R1: 100k 1%, RevK:R_0603, symbol Device:R
- removed R2: 30k 1%, RevK:R_0603, symbol Device:R
- removed U1: LMR16006XDDCR, RevK:SOT-23-Thin-6-Reg, symbol RevK:LMR16006XDDCR
Other:
- moved on the sheet: D1, R1, R2, R3
