File: PCB/Reference/Reference.kicad_pcb (KiCad board)
At the start: 2 copper layers, 10.2 x 12.7 mm, 10 parts, among them J1 Conn_01x04, U1 LMR16006XDDCR

Commit message: Add new reg, and tidy
Parts:
- added C4: 10uF 50V, RevK:C_0603_, F.Cu at (169.8, 62.9)
- added C5: 10uF 6.3V, RevK:C_0603_, F.Cu at (174.8, 62.9)
- added C6: 100nF, RevK:C_0603_, F.Cu at (172.3, 63.6)
- added L2: 10uH, RevK:L_4x4_, F.Cu at (172.3, 66.2)
- added R3: 124k, RevK:R_0402_, F.Cu at (172.3, 59.7)
- added R4: 40k2, RevK:R_0402_, F.Cu at (174.6, 60.8)
- added R5: 1M, RevK:R_0402_, F.Cu at (170.0, 60.8)
- added U2: MD8942, RevK:SOT-23-6-MD8942, F.Cu at (172.3, 61.6)
Routing:
- net GND: vias 1 -> 2
Other:
- board size 10.2 x 12.7 mm -> 24.2 x 12.7 mm
- board text added: "${CURRENT_DATE}"
- board text removed: "${DATE}"

Commit message: Tidy
Parts:
- added D2: RGB, RevK:LED-RGB-1.6x1.6, F.Cu at (145.4, 49.3)
- added FID1: Fiducial, Fiducial:Fiducial_1mm_Mask2mm, F.Cu at (110.0, 32.9)
- added FID2: Fiducial, Fiducial:Fiducial_1mm_Mask2mm, F.Cu at (160.0, 32.9)
- added FID3: Fiducial, Fiducial:Fiducial_1mm_Mask2mm, F.Cu at (160.0, 97.2)
- added FID4: Fiducial, Fiducial:Fiducial_1mm_Mask2mm, F.Cu at (110.0, 97.2)
- added FID5: Fiducial, Fiducial:Fiducial_1mm_Mask2mm, B.Cu at (110.0, 97.2)
- added FID6: Fiducial, Fiducial:Fiducial_1mm_Mask2mm, B.Cu at (160.0, 97.2)
- added FID7: Fiducial, Fiducial:Fiducial_1mm_Mask2mm, B.Cu at (110.0, 32.9)
- added FID8: Fiducial, Fiducial:Fiducial_1mm_Mask2mm, B.Cu at (160.0, 32.9)
- added H1: MountingHole, MountingHole:MountingHole_2mm, F.Cu at (106.0, 40.0)
- added H2: MountingHole, MountingHole:MountingHole_2mm, F.Cu at (165.0, 40.0)
- added H3: MountingHole, MountingHole:MountingHole_2mm, F.Cu at (105.0, 90.0)
- added H4: MountingHole, MountingHole:MountingHole_2mm, F.Cu at (165.0, 90.0)
- added R6: 680R, RevK:R_0402, F.Cu at (143.4, 49.3)
- added R7: 2K, RevK:R_0402, F.Cu at (143.4, 48.3)
- added R8: 220R, RevK:R_0402, F.Cu at (143.4, 50.3)
- added U3: Barcode, RevK:EAN-5060634238069, F.Cu at (118.1, 13.5)
- added U4: Barcode, RevK:EAN-5060634238069, B.Cu at (154.9, 13.9)
- moved C4 38.0 mm to (136.2, 45.2)
- moved C5 38.0 mm to (141.2, 45.2)
- moved C6 38.0 mm to (138.7, 45.9)
- moved L2 38.0 mm to (138.7, 48.5)
- moved R3 38.0 mm to (138.7, 42.0)
- moved U2 38.0 mm to (138.7, 43.9)
- moved U1 38.0 mm to (127.0, 44.7)
- moved C1 38.0 mm to (124.9, 44.9)
- moved C2 38.0 mm to (126.1, 48.2)
- moved C3 38.0 mm to (132.4, 48.2)
- moved D1 38.0 mm to (129.2, 47.8)
- moved J1 38.0 mm to (129.0, 52.1)
- moved L1 38.0 mm to (130.9, 44.7)
- moved Logo1 38.0 mm to (128.4, 43.8)
- moved R1 38.0 mm to (132.5, 42.0)
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Routing:
- net +3.3V: track 0.00 -> 5.77 mm
- net Net-(D2-RK): track 0.00 -> 2.34 mm
- net Net-(D2-BK): track 0.00 -> 1.10 mm
- net Net-(D2-GK): track 0.00 -> 1.09 mm
Other:
- board size 24.2 x 12.7 mm -> 70 x 70 mm
- board text added: "A"
- board text added: "B"
- board text added: "PCB-USBA"
- board text added: "This is an assembled printed circuit board. This is a component, with no case or leads. Snap off any extra blank panels. Use this part for your own projects as you wish. Made in China for Andrews & Arnold Ltd."
- board text added: "USB_A"
- board text added: "generic.revk.uk"

Commit message: Hole
Parts:
- moved H1 1.00 mm to (105.0, 40.0)
Changed lines of the file:
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@@
   )
   (footprint "MountingHole:MountingHole_2mm" (layer "F.Cu")
-    (at 106 40)
+    (at 105 40)
     (descr "Mounting Hole 2mm, no annular")
     (tags "mounting hole 2mm no annular")

Commit message: Tidy
Parts:
- removed H1, H2, H3, H4: MountingHole, MountingHole:MountingHole_2mm
- removed U4: Barcode, RevK:EAN-5060634238069
- U3: moved to B.Cu
- moved U3 69.7 mm to (153.5, 73.5), turned to 180 degrees
- moved FID1 5.00 mm to (105.0, 32.9)
- moved FID2 5.00 mm to (165.0, 32.9)
- moved FID3 5.00 mm to (165.0, 97.2)
- moved FID4 5.00 mm to (105.0, 97.2)
- moved FID5 5.00 mm to (105.0, 97.2)
- moved FID6 5.00 mm to (165.0, 97.2)
- moved FID7 5.00 mm to (105.0, 32.9)
- moved FID8 5.00 mm to (165.0, 32.9)
Other:
- board text removed: "A"
- board text removed: "B"

Commit message: logo
Other:
- board text added: "A"
- board text added: "B"
- board text added: "®"

Commit message: PCB templatge
Parts:
- removed FID1, FID2, FID3, FID4, FID5, FID6, FID7, FID8: Fiducial, Fiducial:Fiducial_1mm_Mask2mm
- added C7: 0.1uF, RevK:C_0402, F.Cu at (142.0, 60.4)
- added PCB1: 70x70, RevK:PCB7070, F.Cu at (135.0, 65.0)
- added R9: 4k7, RevK:R_0402, F.Cu at (139.4, 60.4)
- added U4: CH340X, RevK:CH340X, F.Cu at (141.3, 57.4)
- moved U3 9.45 mm to (153.5, 64.0)
Routing:
- net +3.3V: track 5.77 -> 23.7 mm
- net BOOT: track 0.00 -> 4.41 mm
Other:
- board text added: "?.revk.uk"
- board text added: "PCB-?"
- board text removed: "PCB-USBA"
- board text removed: "generic.revk.uk"

Commit message: Tweak
Parts:
- moved C7 5.15 mm to (141.3, 55.3), turned to 180 degrees
- moved R9 2.11 mm to (141.3, 59.5)
Connections:
- R9 pad 1: +3.3V -> Net-(U4-~{CTS})
- U4 pad 5: GND -> Net-(U4-~{CTS})
Routing:
- net +3.3V: track 23.7 -> 20.0 mm
- net BOOT: track 4.41 -> 2.13 mm
- net Net-(U4-~{CTS}): track 0.00 -> 2.17 mm
Changed lines of the file:
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@@
   (net 23 "I")
   (net 24 "O")
+  (net 25 "Net-(U4-~{CTS})")
   (footprint "RevK:C_0603_" (layer "F.Cu")
     (at 124.87 44.91 90)
@@
   )
   (footprint "RevK:C_0402" (layer "F.Cu")
-    (at 142 60.4)
+    (at 141.3 55.3 180)
     (property "Sheetfile" "Reference.kicad_sch")
     (property "Sheetname" "")
@@
     (property "ki_keywords" "cap capacitor")
     (attr smd)
-    (fp_text reference "C7" (at 0.4 -0.9 unlocked) (layer "F.SilkS") hide
+    (fp_text reference "C7" (at 0.4 -0.9 180 unlocked) (layer "F.SilkS") hide
         (effects (font (size 1 1) (thickness 0.15)))
     )
-    (fp_text value "0.1uF" (at 0 1.1 unlocked) (layer "F.Fab") hide
+    (fp_text value "0.1uF" (at 0 1.1 180 unlocked) (layer "F.Fab") hide
         (effects (font (size 1 1) (thickness 0.15)))
     )
-    (fp_text user "${VALUE}" (at 0 0 unlocked) (layer "F.Fab")
+    (fp_text user "${VALUE}" (at 0 0 180 unlocked) (layer "F.Fab")
         (effects (font (size 0.3 0.3) (thickness 0.05)))
     )
@@
     (fp_line (start 0.75 0.35) (end -0.75 0.35)
       (stroke (width 0.1) (type default)) (layer "F.Fab"))
-    (pad "1" smd roundrect (at -0.5 0) (size 0.54 0.64) (layers "F.Cu" "F.Paste" "F.Mask") (roundrect_rratio 0.25)
+    (pad "1" smd roundrect (at -0.5 0 180) (size 0.54 0.64) (layers "F.Cu" "F.Paste" "F.Mask") (roundrect_rratio 0.25)
       (net 12 "+3.3V") (pintype "passive"))
-    (pad "2" smd roundrect (at 0.5 0) (size 0.54 0.64) (layers "F.Cu" "F.Paste" "F.Mask") (roundrect_rratio 0.25)
+    (pad "2" smd roundrect (at 0.5 0 180) (size 0.54 0.64) (layers "F.Cu" "F.Paste" "F.Mask") (roundrect_rratio 0.25)
       (net 4 "GND") (pintype "passive"))
     (model "${KICAD6_3DMODEL_DIR}/Capacitor_SMD.3dshapes/C_0402_1005Metric.wrl"
@@
   )
   (footprint "RevK:R_0402" (layer "F.Cu")
-    (at 139.39 60.39)
+    (at 141.3 59.5)
     (property "Sheetfile" "Reference.kicad_sch")
     (property "Sheetname" "")
@@
       (stroke (width 0.12) (type solid)) (fill none) (layer "Cmts.User"))
     (pad "1" smd roundrect (at -0.5 0) (size 0.54 0.64) (layers "F.Cu" "F.Paste" "F.Mask") (roundrect_rratio 0.25)
-      (net 12 "+3.3V") (pintype "passive"))
+      (net 25 "Net-(U4-~{CTS})") (pintype "passive"))
     (pad "2" smd roundrect (at 0.5 0) (size 0.54 0.64) (layers "F.Cu" "F.Paste" "F.Mask") (roundrect_rratio 0.25)
       (net 19 "BOOT") (pintype "passive"))
@@
     (descr "10-Lead Plastic Micro Small Outline Package (MS) [MSOP] (see Microchip Packaging Specification 00000049BS.pdf)")
     (tags "SSOP 0.5")
-    (property "JLCPCB Rotation Offset" "90")
+    (property "JLCPCB Rotation Offset" "-90")
     (property "LCSC Part #" "C3035748")
     (property "Sheetfile" "Reference.kicad_sch")
@@
       (net 22 "EN") (pinfunction "~{RTS}") (pintype "output"))
     (pad "5" smd rect (at -2.2 1) (size 1 0.3) (layers "F.Cu" "F.Paste" "F.Mask")
-      (net 4 "GND") (pinfunction "~{CTS}") (pintype "input"))
+      (net 25 "Net-(U4-~{CTS})") (pinfunction "~{CTS}") (pintype "input"))
     (pad "6" smd rect (at 2.2 1) (size 1 0.3) (layers "F.Cu" "F.Paste" "F.Mask")
       (net 19 "BOOT") (pinfunction "TNOW/~{DTR}") (pintype "output"))
@@
   (gr_line (start 126.42 52.96) (end 126.42 51.34)
     (stroke (width 0.5) (type solid)) (layer "F.Mask"))
+  (gr_line (start 100 90) (end 170 90)
+    (stroke (width 0.1) (type default)) (layer "User.1"))
+  (gr_line (start 100 40) (end 170 40)
+    (stroke (width 0.1) (type default)) (layer "User.1"))
   (gr_text "A" (at 109.52 79.05) (layer "B.SilkS")
     (effects (font (face "AJK") (size 8 8) (thickness 0.15)) (justify mirror))
@@
   (via (at 135 51.9) (size 0.8) (drill 0.4) (layers "F.Cu" "B.Cu") (free) (net 4))
   (arc (start 126.9755 42.7505) (mid 126.755684 42.219816) (end 126.225 42) (width 0.2) (layer "F.Cu") (net 4))
-  (segment (start 139.4005 60.9005) (end 138.89 60.39) (width 0.127) (layer "F.Cu") (net 12))
-  (segment (start 138.89 60.39) (end 141.375 57.905) (width 0.127) (layer "F.Cu") (net 12))
+  (segment (start 142.905 56.405) (end 143.48 56.405) (width 0.127) (layer "F.Cu") (net 12))
+  (segment (start 144.107 57.905) (end 143.48 57.905) (width 0.127) (layer "F.Cu") (net 12))
   (segment (start 143.48 56.405) (end 146.3155 53.5695) (width 0.127) (layer "F.Cu") (net 12))
   (segment (start 146.3155 48.9655) (end 145.85 48.5) (width 0.127) (layer "F.Cu") (net 12))
-  (segment (start 141.375 57.905) (end 143.48 57.905) (width 0.127) (layer "F.Cu") (net 12))
-  (segment (start 140.9995 60.9005) (end 139.4005 60.9005) (width 0.127) (layer "F.Cu") (net 12))
+  (segment (start 144.1705 57.8415) (end 144.107 57.905) (width 0.127) (layer "F.Cu") (net 12))
   (segment (start 141.2 45.975) (end 143.481 45.975) (width 0.127) (layer "F.Cu") (net 12))
+  (segment (start 141.8 55.3) (end 142.905 56.405) (width 0.127) (layer "F.Cu") (net 12))
+  (segment (start 144.1705 56.4685) (end 144.1705 57.8415) (width 0.127) (layer "F.Cu") (net 12))
   (segment (start 146.3155 53.5695) (end 146.3155 48.9655) (width 0.127) (layer "F.Cu") (net 12))
-  (segment (start 141.5 60.4) (end 140.9995 60.9005) (width 0.127) (layer "F.Cu") (net 12))
+  (segment (start 144.107 56.405) (end 144.1705 56.4685) (width 0.127) (layer "F.Cu") (net 12))
+  (segment (start 143.48 56.405) (end 144.107 56.405) (width 0.127) (layer "F.Cu") (net 12))
   (segment (start 143.481 45.975) (end 145.739691 48.233691) (width 0.127) (layer "F.Cu") (net 12))
   (arc (start 145.739691 48.233691) (mid 145.821331 48.355874) (end 145.85 48.5) (width 0.127) (layer "F.Cu") (net 12))
@@
   (segment (start 143.9 50.3) (end 144.467158 50.3) (width 0.127) (layer "F.Cu") (net 15))
   (arc (start 144.467158 50.3) (mid 144.72847 50.248022) (end 144.95 50.1) (width 0.127) (layer "F.Cu") (net 15))
-  (segment (start 141.875 58.405) (end 143.48 58.405) (width 0.127) (layer "F.Cu") (net 19))
-  (segment (start 139.89 60.39) (end 141.875 58.405) (width 0.127) (layer "F.Cu") (net 19))
+  (segment (start 142.385 59.5) (end 143.48 58.405) (width 0.127) (layer "F.Cu") (net 19))
+  (segment (start 141.8 59.5) (end 142.385 59.5) (width 0.127) (layer "F.Cu") (net 19))
+  (segment (start 140.175 59.5) (end 139.08 58.405) (width 0.127) (layer "F.Cu") (net 25))
+  (segment (start 140.8 59.5) (end 140.175 59.5) (width 0.127) (layer "F.Cu") (net 25))
   (zone (net 4) (net_name "GND") (layers "F&B.Cu") (hatch edge 0.508)
     (connect_pads (clearance 0.125))

Commit message: VCut
Parts:
- added V1: ~, RevK:VCUT70, F.Cu at (135.0, 42.5)
- added V2: ~, RevK:VCUT70, F.Cu at (135.0, 89.0)
Other:
- board text added: "${TITLE}"
- board text removed: "PCB-?"
